File: examples/unoq-power-shield/pre_route.kicad_pcb (KiCad board)
At the start: 4 copper layers, 53.3 x 68.6 mm, 56 parts, among them J1 VIN 7-24V, J10 UNO PWR, J11 UNO ANALOG, J12 UNO D0-D7, J13 UNO D8-SCL, J2 5V OUT, J3 Qwiic, J4 Qwiic, J5 5V IO, Q1 BSS138LT1G, Q2 BSS138LT1G, Q3 BSS138LT1G, Q4 BSS138LT1G, Q5 AO4407A, U1 TPS54331DDAR, U2 INA226AIDGSR

Commit message: Example board signed off pre-order; add the your-own-board walkthrough
Example (unoq-power-shield), placement/routing rounds to sign-off:
- Final state: 0 unconnected and 0 clearance violations across 5
  identical DRC runs; checker 14 passed / 0 failed; ERC clean; all 24
  JLC BOM lines verified in stock. The 17 residual DRC items (3 kinds)
  are each explained in rev-1-plan.md's new ledger - Qwiic edge pads,
  UNO form-factor header/hole adjacency, courtyard grazes.
- The two structural fixes that ended the recurring PH-past-FB
  clearance cluster: the VIN pour now stops LEFT of U1's pad column
  (as fixed DSN copper it walled off the east corridor and forced PH
  under the chip), and the FB divider + COMP network moved from north
  (y=31-34) to a topology-ordered row south of U1 - FB drops straight
  onto R6/R5 from pin 5, COMP hooks east around the corner onto R7/C7,
  rotations chosen so each pad's net faces its incoming track.
- U2 (MSOP-10) fanout: fan out ONLY pad 7 (GND, plane-fed) via
  skip_pads. A full fanout of a 0.5 mm-pitch part self-blocks: each
  ring via sits one pad pitch from its neighbour's stub, inside the
  0.15 mm clearance at any legal via size (min via 0.5 + min track
  0.2 lands exactly on the pass-a-neighbour bound, and equality
  fails). Alone, the one via that matters fits. Rationale in
  board.toml.
- D3's 5V pad was a dead island (no same-net surface neighbour):
  bonded with a concentric thermal via to the In2 plane.
- Clearance regime settled: netclass clearance IS the DRC constraint
  (0.15 - the MSOP's own 0.2 mm pad gaps must not self-flag);
  completion/astar at 0.16; export_dsn bumps DSN clearances +10 um so
  routed gaps clear the constraint with margin. apply_netclasses
  re-enforces the class clearance from [route].clearance_mm every run.
- bom.csv: 24 lines, every LCSC code verified in stock 2026-08-30.

Pipeline fixes the example paid for:
- export_dsn: +10 um router margin over the DRC constraint;
  class-name comma sanit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
Parts:
- moved C6 14.8 mm to (152.3, 121.8), turned to 90 degrees
- moved C7 14.7 mm to (150.3, 121.8), turned to -90 degrees
- moved R7 14.7 mm to (148.3, 121.8), turned to -90 degrees
- moved J5 14.7 mm to (151.8, 84.3)
- moved R6 14.0 mm to (144.3, 121.8), turned to -90 degrees
- moved R4 13.5 mm to (134.8, 115.8), turned to 90 degrees
- moved R5 11.8 mm to (146.3, 121.8), turned to 90 degrees
- moved C4 10.7 mm to (141.8, 112.8)
- moved D1 10.0 mm to (147.8, 112.8)
- moved R3 8.51 mm to (134.8, 119.3), turned to 90 degrees
- moved R17 5.02 mm to (168.8, 103.8)
- moved R18 5.02 mm to (168.8, 101.3)
- moved R19 5.02 mm to (168.8, 98.8)
- moved D3 5.00 mm to (164.8, 101.3)
- moved C8 2.50 mm to (156.8, 121.3)
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Routing:
- net GND: track 0.00 -> 1.20 mm, vias 8 -> 5
- net 5V: vias 0 -> 1
- added copper zone on F.Cu, net VIN_PROT
- removed copper zone on B.Cu, net GND
- removed copper zone on F.Cu, net GND
