File: examples/unoq-power-shield/unoq-power-shield.kicad_pcb (KiCad board)
At the start: 4 copper layers, 53.3 x 68.6 mm, 56 parts, among them J1 VIN 7-24V, J10 UNO PWR, J11 UNO ANALOG, J12 UNO D0-D7, J13 UNO D8-SCL, J2 5V OUT, J3 Qwiic, J4 Qwiic, J5 5V IO, Q1 BSS138LT1G, Q2 BSS138LT1G, Q3 BSS138LT1G, Q4 BSS138LT1G, Q5 AO4407A, U1 TPS54331DDAR, U2 INA226AIDGSR

Commit message: Prove the schematic humans review is the board that ships
Reviewers open the KiCad project, so it has to be the exact board in the
fab package, including every post-route pass's changes, not a rebuild
that looks the same. Two gaps made that unprovable:

- kct create-pcb wrote footprints with no symbol links, no library
  nickname and no DNP flag. KiCad saw two unrelated documents: 61
  parity items on the example, no cross-probing, and F8 proposing to
  delete every placed part.
- Nothing checked the final board against the schematic. Post-route
  passes set nets on copper they create, and those nets were never
  checked.

New:
- link_schematic (end of build): links each footprint to its symbol,
  copies DNP, and writes fp/sym-lib-table. Marks the holes and fiducials
  board.toml declares as "Not in schematic" and refuses any other
  footprint that has no symbol.
- check_parity (make parity; export_fab refuses without it): runs on the
  final board. KiCad schematic parity; an independent eeschema-netlist
  vs pcbnew-pads diff; DRC x5 failing on shorts or unconnected copper.
  A board-only footprint must be declared and carry no net.
- validate_gerbers --kicad-netlist: X2 pad nets in the plotted copper
  vs the schematic.
- release / verify_release: freeze project + evidence + fab package
  under release/rev-N with hashes; verify re-exports from the released
  board and requires the same package.
- test_parity: 8 ways a pass could damage a board (re-netted pad,
  stray part, shorting track, hidden part, netted hole, value, lost
  link, dropped part); the gate must fail on every one.

Example board: link_schematic applied to the routed board and snapshot.
Diff is metadata only. Gerbers, drill, pos and JLC BOM/CPL re-export
identical apart from dates. All gates pass in KiCad 10.0.5.

Co-Authored-By: Claude Opus 5.5 <noreply@anthropic.com>
Claude-Session: https://claude.ai/code/session_0128ZKZjfVhgiCb6AU4xS1NJ
Parts:
- C1, C2, C8, C9: footprint C_1206_3216Metric -> unoq_power_shield:C_1206_3216Metric
- C10, C3, C4, C5, C6, C7: footprint C_0603_1608Metric -> unoq_power_shield:C_0603_1608Metric
- D1: footprint D_SMA -> unoq_power_shield:D_SMA
- D2: footprint D_SOD-123 -> unoq_power_shield:D_SOD-123
- D3: footprint XL1615RGBC -> unoq_power_shield:XL1615RGBC
- J1, J2: footprint KF301_5.0_2P -> unoq_power_shield:KF301_5.0_2P
- J10, J12: footprint PinHeader_1x08_P2.54mm_Vertical -> unoq_power_shield:PinHeader_1x08_P2.54mm_Vertical
- J11, J5: footprint PinHeader_1x06_P2.54mm_Vertical -> unoq_power_shield:PinHeader_1x06_P2.54mm_Vertical
- J13: footprint PinHeader_1x10_P2.54mm_Vertical -> unoq_power_shield:PinHeader_1x10_P2.54mm_Vertical
- J3, J4: footprint JST_SH_SM04B-SRSS-TB_1x04-1MP_P1.00mm_Horizontal -> unoq_power_shield:JST_SH_SM04B-SRSS-TB_1x04-1MP_P1.00mm_Horizontal
- L1: footprint SWPA6045S -> unoq_power_shield:SWPA6045S
- Q1, Q2, Q3, Q4: footprint SOT-23 -> unoq_power_shield:SOT-23
- Q5: footprint SOIC-8_3.9x4.9mm_P1.27mm -> unoq_power_shield:SOIC-8_3.9x4.9mm_P1.27mm
- R1: footprint R_2512_6332Metric -> unoq_power_shield:R_2512_6332Metric
- R10, R11, R12, R13, R14, R15, R16, R17, R18, R19, R2, R3, R4, R5, R6, R7, R8, R9: footprint R_0603_1608Metric -> unoq_power_shield:R_0603_1608Metric
- U1: footprint TI_SO-PowerPAD-8 -> unoq_power_shield:TI_SO-PowerPAD-8
- U2: footprint MSOP-10_3x3mm_P0.5mm -> unoq_power_shield:MSOP-10_3x3mm_P0.5mm
