File: examples/unoq-power-shield/unoq-power-shield.kicad_pcb (KiCad board)
At the start: 4 copper layers, 53.3 x 68.6 mm, 56 parts, among them J1 VIN 7-24V, J10 UNO PWR, J11 UNO ANALOG, J12 UNO D0-D7, J13 UNO D8-SCL, J2 5V OUT, J3 Qwiic, J4 Qwiic, J5 5V IO, Q1 BSS138LT1G, Q2 BSS138LT1G, Q3 BSS138LT1G, Q4 BSS138LT1G, Q5 AO4407A, U1 TPS54331DDAR, U2 INA226AIDGSR

Commit message: Fix four silk markings printing on pads; check for it in the pass
J5 is the 5 V side of the level shifters (HV1-HV4 + 5V + GND) and its
label read "3.3V LOGIC" — the wrong rail named on the one connector whose
entire purpose is that it is NOT the 3.3 V side. It also printed across
J5's own pads 5 and 6.

The position bug has a reusable cause: a KiCad connector footprint is
anchored at PIN 1, not at its body centre. J5's floorplan (30, 55) puts
pin 1 there and the pads run DOWN to y = 42.35, so a label written at
y = 44 — chosen to sit ~11 mm clear "below" a header assumed to be
centred at 55 — landed between pins 5 and 6.

Adding the check to silk_finish found that two more markings were also on
pads, neither of them noticed by eye:

  * "VIN 7-24V" sat on Q5.3-Q5.6 and D2.1
  * "unoq-power-shield rev1" ran across mounting hole H2's pad

Only "5V 2A" was clean. All four corrected in board.toml, each with the
old coordinates and the reason recorded next to it.

Why nothing caught this: validate_gerbers' silk rule tests containment
inside the outline and nothing else, and silk_finish — which owns a full
pad-mask obstacle model and uses it to reposition all 56 refdeses — only
ever validated [[silk.text]] entries for missing keys and a legal layer,
then placed them literally and treated them as FIXED obstacles that
everything else dodges. The one silk item a human types raw coordinates
for was the one item nothing checked. It now tests every declared marking
against the pad mask openings and warns, naming the board.toml entry.
Warning, not failure: the pass cannot know a better position, only that
this one prints badly (a fab clips silk at the mask opening, so ink on a
pad prints broken AND lands on a solderable surface).

Copper was NOT re-routed — silk cannot move copper, and re-rolling
freerouting for a cosmetic fix would risk the signed-off result. Only
silk_finish and export_fab were re-run, and the gerbers prove the claim:
F.Cu, In1.Cu, In2.Cu, B.Cu, Edge.Cuts, bo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
Other:
- board text added: "5V IO"
- board text removed: "3.3V LOGIC"
Changed lines of the file:
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@@
 		(tags "Through hole pin header THT 1x06 2.54mm single row")
 		(property "Reference" "J11"
-			(at 0 15.615 0)
+			(at 4.5 -2.915 0)
 			(layer "F.SilkS")
 			(effects
@@
 		(tags "SOIC SO")
 		(property "Reference" "Q5"
-			(at 5.62175 4.345 0)
+			(at -1.8 3.845 0)
 			(layer "F.SilkS")
 			(effects
@@
 		(descr "3.2mm NPTH mounting hole, UNO form factor (positions from the UNO Q drill file T08 block: 4x 3.200 NON_PLATED). 6.5mm courtyard = M3 screw head keep-out, an obstacle the placement optimiser packs around.")
 		(property "Reference" "H3"
-			(at -0.001233 -4.396232 0)
+			(at -4.674214 -0.000001 0)
 			(layer "F.SilkS")
 			(effects
@@
 	)
 	(gr_text "VIN 7-24V"
-		(at 130.78 128.84 0)
+		(at 133.78 131.84 0)
 		(layer "F.SilkS")
 		(effects
@@
 		)
 	)
-	(gr_text "3.3V LOGIC"
-		(at 154.78 95.34 0)
+	(gr_text "5V IO"
+		(at 156.78 91.34 0)
 		(layer "F.SilkS")
 		(effects
@@
 	)
 	(gr_text "unoq-power-shield rev1"
-		(at 148.78 138.14 0)
+		(at 144.28 138.14 0)
 		(layer "F.SilkS")
 		(effects
@@
 	)
 	(group "SILK_MARKINGS"
-		(members "a74dc9b2-2325-43be-ad1b-ed8b9d62a277" "a8384525-c663-4f1e-8247-dca25cebaf7e"
-			"c7c2d5a9-3864-49de-aeca-9844726742d9" "f74285c4-2ccf-4501-8ced-d20e2df4b805"
+		(members "038a8c4b-31a0-414b-988e-ec5cb1423e14" "46f41342-3aef-4249-ac44-c82cc929deb1"
+			"d5398fa5-1110-44a3-855c-d0e6052213bb" "e1c0e168-b249-49f4-9916-048e9088b846"
 		)
 	)

Commit message: Example: rotate J4 to face its edge, rebuild; all gates pass
J4 (Qwiic, SM04B-SRSS-TB) was at rotation 180 with its socket opening
into the board. Floorplan now rotation 0, y 3.2 -> 3.4 so the MP tabs
clear the 0.5 mm edge rule by 0.625 mm; the J4 copper_edge_clearance
ledger entry (a symptom of the rotation) is removed.

Rebuilt from netlist.csv in the pinned container (KiCad 10.0.5,
Freerouting 1.9.0) with the fixed pipeline. make check passes:
ERC 0 errors; pad angles all correct; DRC x5 13 errors, all ledgered,
identical every run, 0 unconnected, no stale entries; check_placement
11/0; validate_gerbers 15/0 with IPC-D-356 = netlist.csv 159/159.
drc_report.json, erc_report.json and img/*.png regenerated from the
rebuilt board. Still unfabricated; stock check and committing the exact
ordered package remain for order time (rev-1-plan.md).

Co-Authored-By: Claude Opus 5.5 <noreply@anthropic.com>
Parts:
- moved J4 0.20 mm to (163.3, 135.9), turned to 0 degrees
Routing:
- net HV1: track 291.8 -> 57.4 mm
- net 3V3_UNO: track 222.6 -> 141.3 mm, vias 5 -> 2
- net ALERT_3V3: track 107.1 -> 54.0 mm, vias 4 -> 1
- net UNO_D11: track 48.9 -> 7.19 mm, vias 2 -> 0
- net HV3: track 78.1 -> 40.5 mm, vias 4 -> 0
- net SCL_3V3: track 155.0 -> 119.0 mm, vias 3 -> 1
- net EN: track 41.7 -> 6.07 mm, vias 5 -> 0
- net LV3: track 43.3 -> 13.3 mm, vias 6 -> 1
- net LV2: track 37.9 -> 13.6 mm, vias 4 -> 1
- net HV2: track 73.8 -> 49.8 mm
- net SS: track 27.9 -> 8.59 mm, vias 4 -> 0
- net COMP: track 25.1 -> 7.36 mm, vias 3 -> 0
- net Q5_GATE: track 34.9 -> 21.3 mm, vias 2 -> 0
- net FB: track 20.3 -> 6.72 mm, vias 5 -> 0
- net LV1: track 27.0 -> 14.2 mm, vias 2 -> 1
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